File: Hardware/InkTime_pcb.brd (EAGLE design)
At the start: 46 x 35 mm, 105 parts, among them IC1 BQ25180YBGR, IC2 RT6160AWSC, IC3 BMA423, IC4 DRV2605YZFR, J1 503480-2400, J2 TC2030-IDC, J4 KH-TYPE-C-16P, Q1 20V/4.2A/52mΩ/1.4W, Q3 SI1308EDL-T1-GE3, U1 NRF52840_QF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

Commit message: Am rezolvat issue-urile din pcb 2d
Parts:
- moved ANT1 1.43 mm to (-20.4, -9.70)
- moved L1 1.20 mm to (-17.2, -8.60)
- moved C22 1.00 mm to (-17.1, -10.6)
- moved C4 1.00 mm to (-17.1, -9.60)
Routing:
- net N$4: track 20.1 -> 21.3 mm
- net GND: track 121.7 -> 122.6 mm, vias 48 -> 49
- added copper zone on layer 1, net GND
- added copper zone on layer 16, net GND
